File: hw/fdcanusb.sch (EAGLE design)
At the start: 37 parts, among them J1 MF-CON-MICROUSB-RIGHT, J3 JST-ZH6SMT_VERT, M1 MOUNT, M2 MOUNT, M3 MOUNT, M4 MOUNT, U1 MF-REG-SOT235-3.3V-300mA, U2 USBLC6-2SC6, U3 TCAN334GSOT23, U4 TLP3317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

Commit message: Update PCB to fdcanusb r2.4  * All components are increased to minimum 0603  * Switch to the SOIC package for the CAN transceiver, which is easier    to get  * Switch to 6mil min space/trace
Parts:
- C10, C3, C4, C5, C6, C7, C9: device mfpassives:CAPACITOR_NP_0402 -> mfpassives:CAPACITOR_NP_0603; MPN MF-CAP-0402-0.1uF -> MF-CAP-0603-0.1uF
- R1, R2, R3, R4: device mfpassives:RESISTOR_0402 -> mfpassives:RESISTOR_0603; MPN MF-RES-0402-220 -> MF-RES-0603-220
- R5: value 100 -> 120; MF (none) -> YAGEO; MPN MF-RES-0805-100 -> RC0603FR-07120RL
- R6: device mfpassives:RESISTOR_0402 -> mfpassives:RESISTOR_0603; MPN MF-RES-0402-330 -> MF-RES-0603-330
- U3: value TCAN334GSOT23 -> TCAN334G; device fdcanusb:TCAN334GSOT23 -> fdcanusb:TCAN334G; MPN TCAN334GDCNT -> TCAN330GDR
Other:
- note added: "mjbots fdcanusb r2.4 (c) 2021 Josh Pieper, jpieper@mjbots.com Licensed under the Apache 2.0 License https://www.apache.org/licenses/LICENSE-2.0"
- note removed: "mjbots fdcanusb r2.3 (c) 2021 Josh Pieper, jpieper@mjbots.com Licensed under the Apache 2.0 License https://www.apache.org/licenses/LICENSE-2.0"
Changed lines of the file:
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@@
 </class>
 <class number="1" name="usb" width="0.3048" drill="0">
-<clearance class="1" value="0.127"/>
+<clearance class="1" value="0.1524"/>
 </class>
 <class number="2" name="can" width="0.2159" drill="0">
-<clearance class="2" value="0.127"/>
+<clearance class="2" value="0.1524"/>
 </class>
 </classes>
@@
 <attribute name="POPULATE" value="1"/>
 </part>
-<part name="U3" library="fdcanusb" deviceset="TCAN334G" device="SOT23">
+<part name="U3" library="fdcanusb" deviceset="TCAN334G" device="" value="TCAN334G">
 <attribute name="MF" value="TI"/>
-<attribute name="MPN" value="TCAN334GDCNT"/>
+<attribute name="MPN" value="TCAN330GDR"/>
 <attribute name="POPULATE" value="1"/>
 </part>
@@
 <part name="GND3" library="supply1" deviceset="GND" device=""/>
 <part name="+3V1" library="supply1" deviceset="+3V3" device=""/>
-<part name="C3" library="mfpassives" deviceset="CAPACITOR_NP" device="_0402" value="0.1uF">
-<attribute name="HOUSEPART" value="YES"/>
-<attribute name="MPN" value="MF-CAP-0402-0.1uF"/>
+<part name="C3" library="mfpassives" deviceset="CAPACITOR_NP" device="_0603" value="0.1uF">
+<attribute name="HOUSEPART" value="YES"/>
+<attribute name="MPN" value="MF-CAP-0603-0.1uF"/>
 </part>
 <part name="J3" library="fdcanusb" deviceset="JST-ZH6" device="SMT_VERT">
@@
 <attribute name="POPULATE" value="1"/>
 </part>
-<part name="C7" library="mfpassives" deviceset="CAPACITOR_NP" device="_0402" value="0.1uF">
-<attribute name="HOUSEPART" value="YES"/>
-<attribute name="MPN" value="MF-CAP-0402-0.1uF"/>
+<part name="C7" library="mfpassives" deviceset="CAPACITOR_NP" device="_0603" value="0.1uF">
+<attribute name="HOUSEPART" value="YES"/>
+<attribute name="MPN" value="MF-CAP-0603-0.1uF"/>
 </part>
 <part name="GND4" library="supply1" deviceset="GND" device=""/>
 <part name="GND5" library="supply1" deviceset="GND" device=""/>
-<part name="C5" library="mfpassives" deviceset="CAPACITOR_NP" device="_0402" value="0.1uF">
-<attribute name="HOUSEPART" value="YES"/>
-<attribute name="MPN" value="MF-CAP-0402-0.1uF"/>
-</part>
-<part name="C6" library="mfpassives" deviceset="CAPACITOR_NP" device="_0402" value="0.1uF">
-<attribute name="HOUSEPART" value="YES"/>
-<attribute name="MPN" value="MF-CAP-0402-0.1uF"/>
-</part>
-<part name="C10" library="mfpassives" deviceset="CAPACITOR_NP" device="_0402" value="0.1uF">
-<attribute name="HOUSEPART" value="YES"/>
-<attribute name="MPN" value="MF-CAP-0402-0.1uF"/>
-</part>
-<part name="C9" library="mfpassives" deviceset="CAPACITOR_NP" device="_0402" value="0.1uF">
-<attribute name="HOUSEPART" value="YES"/>
-<attribute name="MPN" value="MF-CAP-0402-0.1uF"/>
+<part name="C5" library="mfpassives" deviceset="CAPACITOR_NP" device="_0603" value="0.1uF">
+<attribute name="HOUSEPART" value="YES"/>
+<attribute name="MPN" value="MF-CAP-0603-0.1uF"/>
+</part>
+<part name="C6" library="mfpassives" deviceset="CAPACITOR_NP" device="_0603" value="0.1uF">
+<attribute name="HOUSEPART" value="YES"/>
+<attribute name="MPN" value="MF-CAP-0603-0.1uF"/>
+</part>
+<part name="C10" library="mfpassives" deviceset="CAPACITOR_NP" device="_0603" value="0.1uF">
+<attribute name="HOUSEPART" value="YES"/>
+<attribute name="MPN" value="MF-CAP-0603-0.1uF"/>
+</part>
+<part name="C9" library="mfpassives" deviceset="CAPACITOR_NP" device="_0603" value="0.1uF">
+<attribute name="HOUSEPART" value="YES"/>
+<attribute name="MPN" value="MF-CAP-0603-0.1uF"/>
 </part>
 <part name="C8" library="mfpassives" deviceset="CAPACITOR_NP" device="_0603" value="1uF">
@@
 <attribute name="MPN" value="MF-CAP-1206-10uF"/>
 </part>
-<part name="C4" library="mfpassives" deviceset="CAPACITOR_NP" device="_0402" value="0.1uF">
-<attribute name="HOUSEPART" value="YES"/>
-<attribute name="MPN" value="MF-CAP-0402-0.1uF"/>
+<part name="C4" library="mfpassives" deviceset="CAPACITOR_NP" device="_0603" value="0.1uF">
+<attribute name="HOUSEPART" value="YES"/>
+<attribute name="MPN" value="MF-CAP-0603-0.1uF"/>
 </part>
 <part name="GND6" library="supply1" deviceset="GND" device=""/>
@@
 <part name="D2" library="mfleds" deviceset="LED_SINGLE" device="-0603-RED" value="MF-LED-0603-RED"/>
 <part name="D4" library="mfleds" deviceset="LED_SINGLE" device="-0603-RED" value="MF-LED-0603-RED"/>
-<part name="R1" library="mfpassives" deviceset="RESISTOR" device="_0402" value="220">
-<attribute name="MPN" value="MF-RES-0402-220"/>
-</part>
-<part name="R2" library="mfpassives" deviceset="RESISTOR" device="_0402" value="220">
-<attribute name="MPN" value="MF-RES-0402-220"/>
-</part>
-<part name="R3" library="mfpassives" deviceset="RESISTOR" device="_0402" value="220">
-<attribute name="MPN" value="MF-RES-0402-220"/>
-</part>
-<part name="R4" library="mfpassives" deviceset="RESISTOR" device="_0402" value="220">
-<attribute name="MPN" value="MF-RES-0402-220"/>
+<part name="R1" library="mfpassives" deviceset="RESISTOR" device="_0603" value="220">
+<attribute name="MPN" value="MF-RES-0603-220"/>
+</part>
+<part name="R2" library="mfpassives" deviceset="RESISTOR" device="_0603" value="220">
+<attribute name="MPN" value="MF-RES-0603-220"/>
+</part>
+<part name="R3" library="mfpassives" deviceset="RESISTOR" device="_0603" value="220">
+<attribute name="MPN" value="MF-RES-0603-220"/>
+</part>
+<part name="R4" library="mfpassives" deviceset="RESISTOR" device="_0603" value="220">
+<attribute name="MPN" value="MF-RES-0603-220"/>
 </part>
 <part name="GND11" library="supply1" deviceset="GND" device=""/>
@@
 <part name="GND12" library="supply1" deviceset="GND" device=""/>
 <part name="+3V7" library="supply1" deviceset="+3V3" device=""/>
-<part name="R5" library="mfpassives" deviceset="RESISTOR" device="_0805" value="100">
-<attribute name="MPN" value="MF-RES-0805-100"/>
+<part name="R5" library="mfpassives" deviceset="RESISTOR" device="_0805" value="120">
+<attribute name="MF" value="YAGEO"/>
+<attribute name="MPN" value="RC0603FR-07120RL"/>
 </part>
 <part name="U4" library="fdcanusb" deviceset="TLP3317" device="">
@@
 </part>
 <part name="+3V8" library="supply1" deviceset="+3V3" device=""/>
-<part name="R6" library="mfpassives" deviceset="RESISTOR" device="_0402" value="330">
-<attribute name="MPN" value="MF-RES-0402-330"/>
+<part name="R6" library="mfpassives" deviceset="RESISTOR" device="_0603" value="330">
+<attribute name="MPN" value="MF-RES-0603-330"/>
 </part>
 </parts>
@@
 <wire x1="-5.08" y1="-63.5" x2="-5.08" y2="88.9" width="0.1524" layer="90"/>
 <text x="0" y="73.66" size="7.62" layer="90">MOUNTS / POWER</text>
-<text x="-5.08" y="93.98" size="3.81" layer="90">mjbots fdcanusb r2.3
+<text x="-5.08" y="93.98" size="3.81" layer="90">mjbots fdcanusb r2.4
 (c) 2021 Josh Pieper, jpieper@mjbots.com
 Licensed under the Apache 2.0 License
@@
 <attribute name="NAME" x="408.94" y="-21.336" size="1.016" layer="95" font="vector" align="top-left"/>
 <attribute name="VALUE" x="408.94" y="-24.384" size="1.016" layer="96" font="vector"/>
+<attribute name="MF" x="406.4" y="-22.86" size="1.778" layer="96" display="off"/>
 </instance>
 <instance part="U4" gate="A" x="381" y="-35.56" smashed="yes">
