File: hw/can.kicad_sch (KiCad schematic)
At the start: 7 parts, among them J1 Conn_01x03, U2 TCAN1057AEVDRQ1, U3 TLP3317

Commit message: WIP - nearly all routing complete
Connections:
- net CAN_P: now reaches J1.1 (Pin_1), R2.2, U2.7 (CANH)
- net CAN_N: now reaches J1.2 (Pin_2), U2.6 (CANL), U3.4
Changed lines of the file:
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@@
     (stroke (width 0) (type default))
+  )
+  (label "CAN_P" (at 162.56 73.66 0) (fields_autoplaced)
+    (effects (font (size 1.27 1.27)) (justify left bottom))
+  )
+  (label "CAN_N" (at 163.83 88.9 0) (fields_autoplaced)
+    (effects (font (size 1.27 1.27)) (justify left bottom))
   )
   (global_label "GND" (shape input) (at 223.52 97.79 270) (fields_autoplaced)
@@
     (effects (font (size 1.27 1.27)) (justify right))
   )
+  (netclass_flag "" (length 2.54) (shape round) (at 148.59 88.9 0) (fields_autoplaced)
+    (effects (font (size 1.27 1.27)) (justify left bottom))
+    (property "Netclass" "can" (at 149.1996 86.36 0)
+      (effects (font (size 1.27 1.27) italic) (justify left))
+    )
+  )
+  (netclass_flag "" (length 2.54) (shape round) (at 148.59 73.66 0) (fields_autoplaced)
+    (effects (font (size 1.27 1.27)) (justify left bottom))
+    (property "Netclass" "can" (at 149.1996 71.12 0)
+      (effects (font (size 1.27 1.27) italic) (justify left))
+    )
+  )
   (symbol (lib_id "Connector_Generic:Conn_01x03") (at 228.6 82.55 0) (unit 1)

Commit message: Add title block and update rev to r4.2
Other:
- company: (none) -> mjbots Robotic Systems, LLC - info@mjbots.com - 2024
- title: (none) -> mjcanfd-usb-1x r4.2
Changed lines of the file:
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@@
 (kicad_sch (version 20230121) (generator eeschema)
   (paper "A4")
+  (title_block
+    (title "mjcanfd-usb-1x r4.2")
+    (company "mjbots Robotic Systems, LLC - info@mjbots.com - 2024")
+    (comment 1 "Licensed under the Apache 2.0 License")
+  )
   (junction (at 54.61 99.06) (diameter 0) (color 0 0 0 0)
   )
