File: hw/fdcanusb.kicad_sch (KiCad schematic)
At the start: 0 parts

Commit message: WIP - nearly all routing complete
Other:
- sheet LED Debug ports: added LED_CAN_RX, LED_CAN_TX, LED_COM, LED_PWR; removed none
Changed lines of the file:
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@@
+    (stroke (width 0) (type default))
+  )
+  (wire (pts (xy 140.97 76.2) (xy 162.56 76.2))
     (stroke (width 0) (type default))
   )
@@
     (stroke (width 0) (type default))
   )
+  (wire (pts (xy 140.97 68.58) (xy 162.56 68.58))
+    (stroke (width 0) (type default))
+  )
   (wire (pts (xy 67.31 46.99) (xy 88.9 46.99))
+    (stroke (width 0) (type default))
+  )
+  (wire (pts (xy 140.97 72.39) (xy 162.56 72.39))
+    (stroke (width 0) (type default))
+  )
+  (wire (pts (xy 140.97 80.01) (xy 162.56 80.01))
     (stroke (width 0) (type default))
   )
@@
       (effects (font (size 1.27 1.27)) (justify left top))
     )
+    (pin "LED_CAN_TX" input (at 162.56 80.01 180)
+      (effects (font (size 1.27 1.27)) (justify left))
+    )
+    (pin "LED_CAN_RX" input (at 162.56 76.2 180)
+      (effects (font (size 1.27 1.27)) (justify left))
+    )
+    (pin "LED_COM" input (at 162.56 68.58 180)
+      (effects (font (size 1.27 1.27)) (justify left))
+    )
+    (pin "LED_PWR" input (at 162.56 72.39 180)
+      (effects (font (size 1.27 1.27)) (justify left))
+    )
     (instances

Commit message: Add title block and update rev to r4.2
Other:
- company: (none) -> mjbots Robotic Systems, LLC - info@mjbots.com - 2024
- title: (none) -> mjcanfd-usb-1x r4.2
Changed lines of the file:
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@@
 (kicad_sch (version 20230121) (generator eeschema)
   (paper "A4")
+  (title_block
+    (title "mjcanfd-usb-1x r4.2")
+    (company "mjbots Robotic Systems, LLC - info@mjbots.com - 2024")
+    (comment 1 "Licensed under the Apache 2.0 License")
+  )
   (wire (pts (xy 67.31 50.8) (xy 88.9 50.8))
     (stroke (width 0) (type default))
