File: hw/stm32g4.kicad_sch (KiCad schematic)
At the start: 10 parts, among them U3 STM32G474CEU6

Commit message: Set up kicadbom and make a pass at filling in all bom entries
Parts:
- C8: MF (none) -> SAMSUNG
Changed lines of the file:
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@@
+      (effects (font (size 1.27 1.27)) hide)
+    )
+    (property "MF" "SAMSUNG" (at 54.61 156.21 0)
       (effects (font (size 1.27 1.27)) hide)
     )

Commit message: Add title block and update rev to r4.2
Other:
- company: (none) -> mjbots Robotic Systems, LLC - info@mjbots.com - 2024
- title: (none) -> mjcanfd-usb-1x r4.2
Changed lines of the file:
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@@
 (kicad_sch (version 20230121) (generator eeschema)
   (paper "A4")
+  (title_block
+    (title "mjcanfd-usb-1x r4.2")
+    (company "mjbots Robotic Systems, LLC - info@mjbots.com - 2024")
+    (comment 1 "Licensed under the Apache 2.0 License")
+  )
   (junction (at 128.27 167.64) (diameter 0) (color 0 0 0 0)
   )
